File: kicad/k1-aioc/k1-aioc.kicad_sch (KiCad schematic)
At the start: 46 parts, among them J1 12401832E402A, J2 Conn_01x07_Male, Q1 BC847BS, U1 MIC5330-SSYML, U2 STM32F373CBTx, Y1 8MHz/20pF

Commit message: Swapping MIC5330 for two TLV1117LV regulators
Since these are easier to solder. Using two regulators to maintain
good PSSR, but this is probably overkill.
Parts:
- removed U1: MIC5330-SSYML, AIOC:Micrel_MLF-8-1EP_2x2mm_P0.5mm_EP0.6x1.2mm, symbol aioc:MIC5330-SSYML
- added FB2: 600R@100MHz, Inductor_SMD:L_0805_2012Metric, symbol Device:FerriteBead
- added U1, U3: TLV1117LV-33, Package_TO_SOT_SMD:SOT-223-3_TabPin2, symbol Regulator_Linear:TLV1117-33
- C3: value 100n -> 4.7u/10V/X5R; LCSC C14663 -> C19666
- renumbered FB2 to FB3
Connections:
- net +3.3VA: now also FB1.2; no longer FB1.1
- net +3V3: now also C5.1, U1.2 (VO); no longer C4.1
- net GND: now also U1.1 (GND), U3.1 (GND)
- net VBUS: now also FB2.1
- net at C3.1: now also FB2.2, U3.3 (VI)
- net VIN: no longer names the net of C6.1, FB3.1
- net VIN: now also U1.3 (VI)
- new net: C4.1, FB1.1, U3.2 (VO)
Other:
- moved on the sheet: C4, C5, C6, FB1, FB3

Commit message: Changing C7 from 4.7uF to 100nF
There is sufficient bulk capacitance on the 3.3V rail but we want
to decouple both VDD inputs of the uC equally.
Parts:
- C7: value 4.7u/10V/X5R -> 100n; LCSC C19666 -> C14663
Changed lines of the file:
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@@
-    (pin "2")
-  )
-  (symbol (lib_id "Device:C") (at 99.06 80.01 0) (unit 1)
-    (in_bom yes) (on_board yes)
-    (property "Reference" "C7" (id 0) (at 92.71 78.74 0)
-      (effects (font (size 1.27 1.27)) (justify left))
-    )
-    (property "Value" "4.7u/10V/X5R" (id 1) (at 81.28 81.28 0)
-      (effects (font (size 1.27 1.27)) (justify left))
-    )
-    (property "Footprint" "Capacitor_SMD:C_0805_2012Metric" (id 2) (at 100.0252 83.82 0)
-      (effects (font (size 1.27 1.27)) hide)
-    )
-    (property "Datasheet" "~" (id 3) (at 99.06 80.01 0)
-      (effects (font (size 1.27 1.27)) hide)
-    )
-    (property "LCSC" "C19666" (id 4) (at 102.87 78.7399 0)
-      (effects (font (size 1.27 1.27)) hide)
-    )
-    (pin "1")
     (pin "2")
   )
@@
     (pin "1")
   )
+  (symbol (lib_id "Device:C") (at 99.06 80.01 0) (mirror y) (unit 1)
+    (in_bom yes) (on_board yes)
+    (property "Reference" "C7" (id 0) (at 102.87 78.7399 0)
+      (effects (font (size 1.27 1.27)) (justify right))
+    )
+    (property "Value" "100n" (id 1) (at 102.87 81.2799 0)
+      (effects (font (size 1.27 1.27)) (justify right))
+    )
+    (property "Footprint" "Capacitor_SMD:C_0805_2012Metric" (id 2) (at 98.0948 83.82 0)
+      (effects (font (size 1.27 1.27)) hide)
+    )
+    (property "Datasheet" "~" (id 3) (at 99.06 80.01 0)
+      (effects (font (size 1.27 1.27)) hide)
+    )
+    (property "LCSC" "C14663" (id 4) (at 95.25 78.7399 0)
+      (effects (font (size 1.27 1.27)) hide)
+    )
+    (pin "1")
+    (pin "2")
+  )
   (symbol (lib_id "power:GND") (at 138.43 52.705 0) (unit 1)
     (in_bom yes) (on_board yes) (fields_autoplaced)
@@
       (reference "C6") (unit 1) (value "4.7u/10V/X5R") (footprint "Capacitor_SMD:C_0805_2012Metric")
     )
-    (path "/aa377a76-cfcf-416f-a662-3566a7ec9a35"
-      (reference "C7") (unit 1) (value "4.7u/10V/X5R") (footprint "Capacitor_SMD:C_0805_2012Metric")
+    (path "/c823c7d5-5bc4-45dc-9607-ac00aa8461d5"
+      (reference "C7") (unit 1) (value "100n") (footprint "Capacitor_SMD:C_0805_2012Metric")
     )
     (path "/e2eb509f-1350-430f-9b40-b0b3d2b9374c"

Commit message: Removing tooling holes
Parts:
- removed H1, H2: ToolingHole, AIOC:TOOLING-HOLE, symbol Mechanical:MountingHole
Changed lines of the file:
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@@
     (pin "1")
-  )
-  (symbol (lib_id "Mechanical:MountingHole") (at 19.05 190.5 0) (unit 1)
-    (in_bom no) (on_board yes) (fields_autoplaced)
-    (property "Reference" "H1" (id 0) (at 21.59 189.2299 0)
-      (effects (font (size 1.27 1.27)) (justify left))
-    )
-    (property "Value" "ToolingHole" (id 1) (at 21.59 191.7699 0)
-      (effects (font (size 1.27 1.27)) (justify left))
-    )
-    (property "Footprint" "AIOC:TOOLING-HOLE" (id 2) (at 19.05 190.5 0)
-      (effects (font (size 1.27 1.27)) hide)
-    )
-    (property "Datasheet" "~" (id 3) (at 19.05 190.5 0)
-      (effects (font (size 1.27 1.27)) hide)
-    )
   )
   (symbol (lib_id "power:GND") (at 99.06 86.36 0) (mirror y) (unit 1)
@@
     (pin "2")
   )
-  (symbol (lib_id "Mechanical:MountingHole") (at 39.37 190.5 0) (unit 1)
-    (in_bom no) (on_board yes) (fields_autoplaced)
-    (property "Reference" "H2" (id 0) (at 41.91 189.2299 0)
-      (effects (font (size 1.27 1.27)) (justify left))
-    )
-    (property "Value" "ToolingHole" (id 1) (at 41.91 191.7699 0)
-      (effects (font (size 1.27 1.27)) (justify left))
-    )
-    (property "Footprint" "AIOC:TOOLING-HOLE" (id 2) (at 39.37 190.5 0)
-      (effects (font (size 1.27 1.27)) hide)
-    )
-    (property "Datasheet" "~" (id 3) (at 39.37 190.5 0)
-      (effects (font (size 1.27 1.27)) hide)
-    )
-  )
   (symbol (lib_id "Regulator_Linear:TLV1117-33") (at 124.46 45.085 0) (unit 1)
     (in_bom yes) (on_board yes) (fields_autoplaced)
@@
       (reference "FB3") (unit 1) (value "600R@100MHz") (footprint "Inductor_SMD:L_0805_2012Metric")
     )
-    (path "/098bba9b-ee08-4339-943b-7dd4169e891d"
-      (reference "H1") (unit 1) (value "ToolingHole") (footprint "AIOC:TOOLING-HOLE")
-    )
-    (path "/ba24aaa2-cdf6-43f8-bf42-f4a3c365b43c"
-      (reference "H2") (unit 1) (value "ToolingHole") (footprint "AIOC:TOOLING-HOLE")
-    )
     (path "/c5b80805-bc26-457d-a1fd-cf6a8b83ea3f"
