File: kicad/k1-aioc/k1-aioc.kicad_sch (KiCad schematic)
At the start: 46 parts, among them J1 12401832E402A, J2 Conn_01x07_Male, Q1 BC847BS, U1 TLV1117LV-33, U2 STM32F373CBTx, U3 TLV1117LV-33, Y1 8MHz/20pF

Commit message: Adding USB isolation
- Isolated 5V DC/DC converter
- ADUM3160 USB Isolator
- 1.5k PU optional (handled by ADUM3160)
Parts:
- added C16, C17: 4.7u/10V/X5R, Capacitor_SMD:C_0805_2012Metric, symbol Device:C
- added C18, C19: 100n, Capacitor_SMD:C_0805_2012Metric, symbol Device:C
- added R18, R19, R21, R22: 24, Resistor_SMD:R_0805_2012Metric, symbol Device:R
- added R20: 5.1K, Resistor_SMD:R_0805_2012Metric, symbol Device:R
- added U4: CRE1S0505SC, Converter_DCDC:Converter_DCDC_Murata_CRE1xxxxxxSC_THT, symbol Regulator_Switching:CRE1S0505SC
- added U5: ADUM3160, Package_SO:SOIC-16W_7.5x10.3mm_P1.27mm, symbol Interface_USB:ADUM3160
Connections:
- net GND: now also C17.2, C19.2, U4.3 (-VOUT), U5.15 (GND2), U5.9 (GND2); no longer J1.A1 (GND), J1.A12 (GND), J1.B1 (GND), J1.B12 (GND), J1.S1 (SHIELD), R6.1, R7.1
- net USB-DN: no longer names the net of J1.A7 (D-), J1.B7 (D-)
- net USB-DN: now also R18.2; no longer U2.32 (PA11)
- net USB-DP: no longer names the net of J1.A6 (D+), J1.B6 (D+)
- net USB-DP: now also R19.2; no longer R1.2, U2.33 (PA12)
- net VBUS: no longer names the net of J1.A4 (VBUS), J1.A9 (VBUS), J1.B4 (VBUS), J1.B9 (VBUS)
- net VBUS: now also C16.1, U4.2 (+VIN), U5.1 (VBUS1); no longer FB2.1, FB3.2
- new net: R21.2, U5.10 (DD+)
- new net: C17.1, FB2.1, FB3.2, U4.4 (+VOUT), U5.16 (VBUS2)
- new net: R22.2, U5.11 (DD-)
- new net: C19.1, R20.2, U5.13 (SPD), U5.14 (VDD2)
- new net: C18.1, U5.3 (VDD1), U5.4 (PDEN), U5.5 (SPU)
- new net: R20.1, U5.12 (PIN)
- new net GNDREF: C16.2, C18.2, J1.A1 (GND), J1.A12 (GND), J1.B1 (GND), J1.B12 (GND), J1.S1 (SHIELD), R6.1, R7.1, U4.1 (-VIN), U5.2 (GND1), U5.8 (GND1)
- new net USB-DN-D: R22.1, U2.32 (PA11)
- new net USB-DN-H: R18.1, U5.6 (UD-)
- new net USB-DP-D: R1.2, R21.1, U2.33 (PA12)
- new net USB-DP-H: R19.1, U5.7 (UD+)
- no-connect marks 0 -> 2
Other:
- note added: "ENUMERATION"
- moved on the sheet: C1, C10, C11, C12, C13, C14, C15, C2, C3, C4, C5, C6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

Commit message: Removing PTT2, swapping Q1
- PTT2 is not required, removing circuitry
- Q1 was dual transistor, replaced with PZT2222A
- 22R --> 24R for Q1 collector (minimizing BOM)
- Cleaned up schematic
Parts:
- removed Q1: BC847BS, Package_TO_SOT_SMD:SOT-363_SC-70-6, symbol Device:Q_Dual_NPN_NPN_E1B1C2E2B2C1
- removed R10: 2.2K, Resistor_SMD:R_0805_2012Metric, symbol Device:R
- removed R12: 22R, Resistor_SMD:R_0805_2012Metric, symbol Device:R
- added Q1: PZT2222A, Package_TO_SOT_SMD:SOT-223-3_TabPin2, symbol Transistor_BJT:PZT2222A
- R13: value 22R -> 24R; LCSC C23345 -> (none)
Connections:
- net GND: now also Q1.3 (E)
- net at FB2.1, FB3.2, U5.16 (VBUS2): no longer C17.1, U4.4 (+VOUT)
- net at R13.2: now also Q1.2 (C)
- net at R11.2: now also Q1.1 (B)
- net PTT2: no longer names the net of U2.10 (PA0)
- new net: C17.1, U4.4 (+VOUT)
Other:
- moved on the sheet: C16, C17, C18, C19, C3, C4, C5, C6, FB1, FB2, FB3, R18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

Commit message: Adding two TRRS jacks for I/O (digirig pinout)
Parts:
- added J3: AUDIO, Connector_Audio:Jack_3.5mm_PJ320E_Horizontal, symbol Connector:AudioJack4
- added J4: CAT, Connector_Audio:Jack_3.5mm_PJ320E_Horizontal, symbol Connector:AudioJack4
- added Q?: PZT2222A, Package_TO_SOT_SMD:SOT-223-3_TabPin2, symbol Transistor_BJT:PZT2222A
Connections:
- net GND: now also J3.S, J4.S
- net RADIO-MIC: now also J3.R1
- net RADIO-SPK: now also J3.T
- net RADIO-TX: now also J4.R1
- net RADIO-RX-PTT1 renamed RADIO-PTT
- net RADIO-PTT: now also J3.R2; no longer R8.1
- new net RADIO-RX: J4.T, R8.1
Other:
- note removed: "K connector consists of two TRS connectors (3.5mm and 2.5mm) spaced 12mm apart Upper connector (2.5mm) T: SPK+ R: TxData (from Radio) S: GND Lower connector (3.5mm) T: +V/PTT2 R: MIC+ S: PTT1/RxData (to Radio)"
- moved on the sheet: C13, R13, R16

Commit message: Adding general purpose input (e.g. use for COS)
Parts:
- removed Q?: PZT2222A, Package_TO_SOT_SMD:SOT-223-3_TabPin2, symbol Transistor_BJT:PZT2222A
- added Q2: PZT2222A, Package_TO_SOT_SMD:SOT-223-3_TabPin2, symbol Transistor_BJT:PZT2222A
- added R10: 24R, Resistor_SMD:R_0805_2012Metric, symbol Device:R
Connections:
- net GND: now also Q2.3 (E)
- net at C17.1, U4.4 (+VOUT): now also FB2.1, FB3.2, U5.16 (VBUS2)
- net at U2.29 (PA8): now also Q2.2 (C)
- net COS: now reaches J4.R2
- net COS: now also R10.1
- new net: Q2.1 (B), R10.2
Other:
- moved on the sheet: C12, C13, J3, R13, R4

Commit message: Removing JLC part numbers for 0603 --> 0805 parts
Parts:
- C1, C2: LCSC C1653 -> (none)
- C10, C13, C14, C16, C17, C3, C4, C5, C6: LCSC C19666 -> (none)
- C11: LCSC C57112 -> (none)
- C12, C15, C18, C19, C7, C8, C9: LCSC C14663 -> (none)
- FB1, FB2, FB3: LCSC C1002 -> (none)
- R1: LCSC C22843 -> (none)
- R11, R14, R5: LCSC C4190 -> (none)
- R15, R4, R8, R9: LCSC C22962 -> (none)
- R16, R20, R3, R6, R7: LCSC C23186 -> (none)
- R2: LCSC C25804 -> (none)
Changed lines of the file:
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@@
       (effects (font (size 1.27 1.27)) hide)
     )
-    (property "LCSC" "C22962" (id 4) (at 180.34 121.92 0)
+    (property "LCSC" "" (id 4) (at 180.34 121.92 0)
       (effects (font (size 1.27 1.27)) hide)
     )
@@
       (effects (font (size 1.27 1.27)) hide)
     )
-    (property "LCSC" "C19666" (id 4) (at 137.16 24.7649 0)
+    (property "LCSC" "" (id 4) (at 137.16 24.7649 0)
       (effects (font (size 1.27 1.27)) hide)
     )
@@
       (effects (font (size 1.27 1.27)) hide)
     )
-    (property "LCSC" "C4190" (id 4) (at 214.63 143.51 0)
+    (property "LCSC" "" (id 4) (at 214.63 143.51 0)
       (effects (font (size 1.27 1.27)) hide)
     )
@@
       (effects (font (size 1.27 1.27)) hide)
     )
-    (property "LCSC" "C22962" (id 4) (at 147.32 160.02 0)
+    (property "LCSC" "" (id 4) (at 147.32 160.02 0)
       (effects (font (size 1.27 1.27)) hide)
     )
@@
       (effects (font (size 1.27 1.27)) hide)
     )
-    (property "LCSC" "C23186" (id 4) (at 78.105 60.3249 0)
+    (property "LCSC" "" (id 4) (at 78.105 60.3249 0)
       (effects (font (size 1.27 1.27)) hide)
     )
@@
       (effects (font (size 1.27 1.27)) hide)
     )
-    (property "LCSC" "C14663" (id 4) (at 220.98 94.6149 0)
+    (property "LCSC" "" (id 4) (at 220.98 94.6149 0)
       (effects (font (size 1.27 1.27)) hide)
     )
@@
       (effects (font (size 1.27 1.27)) hide)
     )
-    (property "LCSC" "C19666" (id 4) (at 107.315 24.7649 0)
+    (property "LCSC" "" (id 4) (at 107.315 24.7649 0)
       (effects (font (size 1.27 1.27)) hide)
     )
@@
       (effects (font (size 1.27 1.27)) hide)
     )
-    (property "LCSC" "C1002" (id 4) (at 245.6942 34.29 0)
+    (property "LCSC" "" (id 4) (at 245.6942 34.29 0)
       (effects (font (size 1.27 1.27)) hide)
     )
@@
       (effects (font (size 1.27 1.27)) hide)
     )
-    (property "LCSC" "C1653" (id 4) (at 58.42 171.45 0)
+    (property "LCSC" "" (id 4) (at 58.42 171.45 0)
       (effects (font (size 1.27 1.27)) hide)
     )
@@
       (effects (font (size 1.27 1.27)) hide)
     )
-    (property "LCSC" "C19666" (id 4) (at 228.6 84.455 0)
+    (property "LCSC" "" (id 4) (at 228.6 84.455 0)
       (effects (font (size 1.27 1.27)) hide)
     )
@@
       (effects (font (size 1.27 1.27)) hide)
     )
-    (property "LCSC" "C1002" (id 4) (at 198.8058 42.545 0)
+    (property "LCSC" "" (id 4) (at 198.8058 42.545 0)
       (effects (font (size 1.27 1.27)) hide)
     )
@@
       (effects (font (size 1.27 1.27)) hide)
     )
-    (property "LCSC" "C19666" (id 4) (at 210.82 29.2099 0)
+    (property "LCSC" "" (id 4) (at 210.82 29.2099 0)
       (effects (font (size 1.27 1.27)) hide)
     )
@@
       (effects (font (size 1.27 1.27)) hide)
     )
-    (property "LCSC" "C1002" (id 4) (at 198.7042 34.29 0)
+    (property "LCSC" "" (id 4) (at 198.7042 34.29 0)
       (effects (font (size 1.27 1.27)) hide)
     )
@@
       (effects (font (size 1.27 1.27)) hide)
     )
-    (property "LCSC" "C22843" (id 4) (at 158.7499 129.54 0)
+    (property "LCSC" "" (id 4) (at 158.7499 129.54 0)
       (effects (font (size 1.27 1.27)) hide)
     )
@@
       (effects (font (size 1.27 1.27)) hide)
     )
-    (property "LCSC" "C19666" (id 4) (at 224.79 142.24 0)
+    (property "LCSC" "" (id 4) (at 224.79 142.24 0)
       (effects (font (size 1.27 1.27)) hide)
     )
@@
       (effects (font (size 1.27 1.27)) hide)
     )
-    (property "LCSC" "C14663" (id 4) (at 174.625 43.8149 0)
+    (property "LCSC" "" (id 4) (at 174.625 43.8149 0)
       (effects (font (size 1.27 1.27)) hide)
     )
@@
       (effects (font (size 1.27 1.27)) hide)
     )
-    (property "LCSC" "C19666" (id 4) (at 156.21 89.5349 0)
+    (property "LCSC" "" (id 4) (at 156.21 89.5349 0)
       (effects (font (size 1.27 1.27)) hide)
     )
@@
       (effects (font (size 1.27 1.27)) hide)
     )
-    (property "LCSC" "C22962" (id 4) (at 184.15 129.54 0)
+    (property "LCSC" "" (id 4) (at 184.15 129.54 0)
       (effects (font (size 1.27 1.27)) hide)
     )
@@
       (effects (font (size 1.27 1.27)) hide)
     )
-    (property "LCSC" "C57112" (id 4) (at 190.5 152.4 0)
+    (property "LCSC" "" (id 4) (at 190.5 152.4 0)
       (effects (font (size 1.27 1.27)) hide)
     )
@@
       (effects (font (size 1.27 1.27)) hide)
     )
-    (property "LCSC" "C23186" (id 4) (at 82.55 60.3249 0)
+    (property "LCSC" "" (id 4) (at 82.55 60.3249 0)
       (effects (font (size 1.27 1.27)) hide)
     )
@@
       (effects (font (size 1.27 1.27)) hide)
     )
-    (property "LCSC" "C4190" (id 4) (at 180.34 100.33 0)
+    (property "LCSC" "" (id 4) (at 180.34 100.33 0)
       (effects (font (size 1.27 1.27)) hide)
     )
@@
       (effects (font (size 1.27 1.27)) hide)
     )
-    (property "LCSC" "C25804" (id 4) (at 182.8799 111.76 0)
+    (property "LCSC" "" (id 4) (at 182.8799 111.76 0)
       (effects (font (size 1.27 1.27)) hide)
     )
@@
       (effects (font (size 1.27 1.27)) hide)
     )
-    (property "LCSC" "C14663" (id 4) (at 87.63 43.8149 0)
+    (property "LCSC" "" (id 4) (at 87.63 43.8149 0)
       (effects (font (size 1.27 1.27)) hide)
     )
@@
       (effects (font (size 1.27 1.27)) hide)
     )
-    (property "LCSC" "C23186" (id 4) (at 199.39 146.0501 0)
+    (property "LCSC" "" (id 4) (at 199.39 146.0501 0)
       (effects (font (size 1.27 1.27)) hide)
     )
@@
       (effects (font (size 1.27 1.27)) hide)
     )
-    (property "LCSC" "C23186" (id 4) (at 204.47 152.3999 0)
+    (property "LCSC" "" (id 4) (at 204.47 152.3999 0)
       (effects (font (size 1.27 1.27)) hide)
     )
@@
       (effects (font (size 1.27 1.27)) hide)
     )
-    (property "LCSC" "C4190" (id 4) (at 78.74 114.2999 0)
+    (property "LCSC" "" (id 4) (at 78.74 114.2999 0)
       (effects (font (size 1.27 1.27)) hide)
     )
@@
       (effects (font (size 1.27 1.27)) hide)
     )
-    (property "LCSC" "C1653" (id 4) (at 87.63 171.4499 0)
+    (property "LCSC" "" (id 4) (at 87.63 171.4499 0)
       (effects (font (size 1.27 1.27)) hide)
     )
@@
       (effects (font (size 1.27 1.27)) hide)
     )
-    (property "LCSC" "C14663" (id 4) (at 95.25 89.5349 0)
+    (property "LCSC" "" (id 4) (at 95.25 89.5349 0)
       (effects (font (size 1.27 1.27)) hide)
     )
@@
       (effects (font (size 1.27 1.27)) hide)
     )
-    (property "LCSC" "C14663" (id 4) (at 69.85 114.2999 0)
+    (property "LCSC" "" (id 4) (at 69.85 114.2999 0)
       (effects (font (size 1.27 1.27)) hide)
     )
@@
       (effects (font (size 1.27 1.27)) hide)
     )
-    (property "LCSC" "C19666" (id 4) (at 238.125 52.7049 0)
+    (property "LCSC" "" (id 4) (at 238.125 52.7049 0)
       (effects (font (size 1.27 1.27)) hide)
     )
@@
       (effects (font (size 1.27 1.27)) hide)
     )
-    (property "LCSC" "C19666" (id 4) (at 210.82 52.7049 0)
+    (property "LCSC" "" (id 4) (at 210.82 52.7049 0)
       (effects (font (size 1.27 1.27)) hide)
     )
@@
       (effects (font (size 1.27 1.27)) hide)
     )
-    (property "LCSC" "C14663" (id 4) (at 106.68 89.5349 0)
+    (property "LCSC" "" (id 4) (at 106.68 89.5349 0)
       (effects (font (size 1.27 1.27)) hide)
     )
@@
       (effects (font (size 1.27 1.27)) hide)
     )
-    (property "LCSC" "C23186" (id 4) (at 137.1601 46.355 0)
+    (property "LCSC" "" (id 4) (at 137.1601 46.355 0)
       (effects (font (size 1.27 1.27)) hide)
     )
@@
       (effects (font (size 1.27 1.27)) hide)
     )
-    (property "LCSC" "C14663" (id 4) (at 137.16 89.5349 0)
+    (property "LCSC" "" (id 4) (at 137.16 89.5349 0)
       (effects (font (size 1.27 1.27)) hide)
     )
@@
       (effects (font (size 1.27 1.27)) hide)
     )
-    (property "LCSC" "C22962" (id 4) (at 209.55 94.6149 0)
+    (property "LCSC" "" (id 4) (at 209.55 94.6149 0)
       (effects (font (size 1.27 1.27)) hide)
     )
@@
       (effects (font (size 1.27 1.27)) hide)
     )
-    (property "LCSC" "C19666" (id 4) (at 238.125 29.2099 0)
-      (effects (font (size 1.27 1.27)) hide)
-    )
+    (property "LCSC" "" (id 4) (at 238.125 29.2099 0)
+      (effects (font (size 1.27 1.27)) hide)
+    )

Commit message: Replacing discrete LEDs with RGB LED (different pins)
Parts:
- removed D1: GREEN, LED_SMD:LED_0603_1608Metric, symbol Device:LED
- removed D2: RED, LED_SMD:LED_0603_1608Metric, symbol Device:LED
- removed D3, D4: N.M., LED_SMD:LED_0603_1608Metric, symbol Device:LED
- added D1: LED_RGBK, LED_SMD:LED_Kingbright_APFA3010_3x1.5mm_Horizontal, symbol Device:LED_RKGB
- added R12, R23: 220R, Resistor_SMD:R_0805_2012Metric, symbol Device:R
Connections:
- net GND: now also D1.2 (K)
- net at R15.1: now also D1.3 (GA)
- net at U2.45 (PB8): no longer R15.2
- net LED_G: now reaches U2.26 (PB14)
- net LED_G: now also R15.2
- net LED_B: now reaches U2.27 (PB15)
- net LED_B: now also R12.2
- net LED_R: now reaches U2.28 (PD8)
- net LED_R: now also R23.2
- new net: D1.4 (BA), R12.1
- new net: D1.1 (RA), R23.1

Commit message: Adding GND point for scope probe
Parts:
- added J5: GND, Connector_PinHeader_2.54mm:PinHeader_1x02_P2.54mm_Vertical, symbol Connector:Conn_01x02_Male
Connections:
- net GND: now also J5.1 (Pin_1), J5.2 (Pin_2)
Changed lines of the file:
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@@
     (rev "1.0")
+  )
+  (junction (at 44.45 154.94) (diameter 0) (color 0 0 0 0)
   )
   (junction (at 123.19 69.215) (diameter 0) (color 0 0 0 0)
@@
     (stroke (width 0) (type default) (color 0 0 0 0))
   )
+  (wire (pts (xy 44.45 152.4) (xy 44.45 154.94))
+    (stroke (width 0) (type default) (color 0 0 0 0))
+  )
   (wire (pts (xy 132.08 51.435) (xy 138.43 51.435))
     (stroke (width 0) (type default) (color 0 0 0 0))
@@
     (stroke (width 0) (type default) (color 0 0 0 0))
   )
+  (wire (pts (xy 44.45 154.94) (xy 44.45 155.575))
+    (stroke (width 0) (type default) (color 0 0 0 0))
+  )
   (wire (pts (xy 228.6 26.67) (xy 234.315 26.67))
     (stroke (width 0) (type default) (color 0 0 0 0))
@@
     (stroke (width 0) (type default) (color 0 0 0 0))
   )
+  (wire (pts (xy 36.83 152.4) (xy 44.45 152.4))
+    (stroke (width 0) (type default) (color 0 0 0 0))
+  )
   (wire (pts (xy 99.06 83.185) (xy 99.06 86.995))
+    (stroke (width 0) (type default) (color 0 0 0 0))
+  )
+  (wire (pts (xy 36.83 154.94) (xy 44.45 154.94))
     (stroke (width 0) (type default) (color 0 0 0 0))
   )
@@
     (pin "1")
   )
+  (symbol (lib_id "Connector:Conn_01x02_Male") (at 31.75 154.94 0) (mirror x) (unit 1)
+    (in_bom yes) (on_board yes)
+    (property "Reference" "J5" (id 0) (at 35.56 146.05 0)
+      (effects (font (size 1.27 1.27)) (justify right))
+    )
+    (property "Value" "GND" (id 1) (at 36.195 148.59 0)
+      (effects (font (size 1.27 1.27)) (justify right))
+    )
+    (property "Footprint" "Connector_PinHeader_2.54mm:PinHeader_1x02_P2.54mm_Vertical" (id 2) (at 31.75 154.94 0)
+      (effects (font (size 1.27 1.27)) hide)
+    )
+    (property "Datasheet" "~" (id 3) (at 31.75 154.94 0)
+      (effects (font (size 1.27 1.27)) hide)
+    )
+    (pin "1")
+    (pin "2")
+  )
   (symbol (lib_id "Device:C") (at 178.435 45.085 0) (mirror y) (unit 1)
     (in_bom yes) (on_board yes)
@@
     (pin "2")
   )
+  (symbol (lib_id "power:GND") (at 44.45 155.575 0) (mirror y) (unit 1)
+    (in_bom yes) (on_board yes) (fields_autoplaced)
+    (property "Reference" "#PWR0135" (id 0) (at 44.45 161.925 0)
+      (effects (font (size 1.27 1.27)) hide)
+    )
+    (property "Value" "GND" (id 1) (at 44.45 160.655 0))
+    (property "Footprint" "" (id 2) (at 44.45 155.575 0)
+      (effects (font (size 1.27 1.27)) hide)
+    )
+    (property "Datasheet" "" (id 3) (at 44.45 155.575 0)
+      (effects (font (size 1.27 1.27)) hide)
+    )
+    (pin "1")
+  )
   (symbol (lib_id "Device:C") (at 207.01 53.975 0) (unit 1)
     (in_bom yes) (on_board yes)
@@
       (reference "#PWR0134") (unit 1) (value "GND") (footprint "")
     )
+    (path "/e01d29eb-83cc-47e6-b20d-2cac1f6f776b"
+      (reference "#PWR0135") (unit 1) (value "GND") (footprint "")
+    )
     (path "/4f4a10d7-b161-42d7-90b7-9b7948641a9a"
       (reference "C1") (unit 1) (value "22p/NP0") (footprint "Capacitor_SMD:C_0805_2012Metric")
@@
       (reference "J4") (unit 1) (value "CAT") (footprint "Connector_Audio:Jack_3.5mm_PJ320E_Horizontal")
     )
+    (path "/761380c9-ed79-45c9-9f6a-cc208bb77421"
+      (reference "J5") (unit 1) (value "GND") (footprint "Connector_PinHeader_2.54mm:PinHeader_1x02_P2.54mm_Vertical")
+    )
     (path "/7976f8cd-bffe-4aeb-a16a-027a2e13ef41"

Commit message: Adding LCSC (and some DIGIKEY) part numbers
Parts:
- C1, C2: LCSC (none) -> C376875
- C10, C13, C14, C16, C17, C3, C4, C5, C6: LCSC (none) -> C5375826
- C11: LCSC (none) -> C237168
- C12, C15, C18, C19, C7, C8, C9: LCSC (none) -> C720961
- D1: DIGIKEY (none) -> 754-2148-1-ND
- FB1, FB2, FB3: LCSC (none) -> C124100
- J1: DIGIKEY (none) -> 12401832E402ACT-ND
- J3, J4: LCSC (none) -> C2939183
- Q1, Q2: LCSC (none) -> C7603308
- R1: LCSC (none) -> C2907216
- R10, R13: LCSC (none) -> C3017901
- R11, R14, R5: LCSC (none) -> C104106
- R12, R15, R23, R4, R8, R9: LCSC (none) -> C3016631
- R16, R20, R3, R6, R7: LCSC (none) -> C104375
- R18, R19, R21, R22: value 24 -> 24R; LCSC (none) -> C3017901
- R2: LCSC (none) -> C3016734
- U1, U3: DIGIKEY (none) -> 296-28778-1-ND; LCSC (none) -> C15578
- U2: DIGIKEY (none) -> 497-17414-ND
- U4: DIGIKEY (none) -> 811-3196-ND; LCSC (none) -> C2912568
- U5: DIGIKEY (none) -> ADUM3160BRWZ-RLCT-ND; LCSC (none) -> C108501
