File: kicad/k1-aioc/k1-aioc.kicad_pcb (KiCad board)
At the start: 2 copper layers, 47.5 x 80 mm, 58 parts, among them J1 12401832E402A, J2 Conn_01x07_Male, J3 AUDIO, J4 CAT, Q1 PZT2222A, Q2 PZT2222A, U1 TLV1117LV-33, U2 STM32F373CBTx, U3 TLV1117LV-33, U4 CRE1S0505SC, U5 ADUM3160, Y1 8MHz/20pF

Commit message: Adding some more via stitching
Routing:
- net GND: vias 196 -> 200
Changed lines of the file:
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@@
   (segment (start 246.425 49.9) (end 246.425 51.675) (width 0.5) (layer "F.Cu") (net 1))
   (via (at 229.4 50.4) (size 0.6) (drill 0.3) (layers "F.Cu" "B.Cu") (free) (net 1))
+  (via (at 217.6 60) (size 0.6) (drill 0.3) (layers "F.Cu" "B.Cu") (free) (net 1))
   (via (at 220.2 65.4) (size 0.6) (drill 0.3) (layers "F.Cu" "B.Cu") (free) (net 1))
   (via (at 243.8 103.8) (size 0.6) (drill 0.3) (layers "F.Cu" "B.Cu") (free) (net 1))
@@
   (via (at 225.4 54) (size 0.6) (drill 0.3) (layers "F.Cu" "B.Cu") (free) (net 1))
   (via (at 210.2 108) (size 0.6) (drill 0.3) (layers "F.Cu" "B.Cu") (free) (net 1))
+  (via (at 215.6 55) (size 0.6) (drill 0.3) (layers "F.Cu" "B.Cu") (free) (net 1))
   (via (at 206.8 64) (size 0.6) (drill 0.3) (layers "F.Cu" "B.Cu") (free) (net 1))
   (via (at 240.6 90.2) (size 0.6) (drill 0.3) (layers "F.Cu" "B.Cu") (free) (net 1))
@@
   (via (at 245 91.5) (size 0.6) (drill 0.3) (layers "F.Cu" "B.Cu") (net 1))
   (via (at 206 87.8) (size 0.6) (drill 0.3) (layers "F.Cu" "B.Cu") (free) (net 1))
+  (via (at 217.6 55) (size 0.6) (drill 0.3) (layers "F.Cu" "B.Cu") (free) (net 1))
   (via (at 217.2 64.8) (size 0.6) (drill 0.3) (layers "F.Cu" "B.Cu") (free) (net 1))
   (via (at 226 104.8) (size 0.6) (drill 0.3) (layers "F.Cu" "B.Cu") (free) (net 1))
@@
   (via (at 206 80.6) (size 0.6) (drill 0.3) (layers "F.Cu" "B.Cu") (free) (net 1))
   (via (at 245.75 60.59375) (size 0.6) (drill 0.3) (layers "F.Cu" "B.Cu") (net 1))
+  (via (at 217.6 57.6) (size 0.6) (drill 0.3) (layers "F.Cu" "B.Cu") (free) (net 1))
   (via (at 219.4 48.2) (size 0.6) (drill 0.3) (layers "F.Cu" "B.Cu") (free) (net 1))
   (via (at 233.4 50.4) (size 0.6) (drill 0.3) (layers "F.Cu" "B.Cu") (free) (net 1))

Commit message: Silk screen: Name, acknowledgement and revision
Other:
- board text added: "HB9UF All-In-One-Box, Rev 1.0, (c) 2024 M. Weyland HB9FRV, based on work by skuep"
Changed lines of the file:
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@@
     (property "Sheetname" "")
     (attr smd)
-    (fp_text reference "C16" (at 0 -2 90) (layer "F.SilkS")
+    (fp_text reference "C16" (at 3.7 0 90) (layer "F.SilkS")
       (effects (font (size 1 1) (thickness 0.15)))
     )
@@
   (gr_arc (start 208.5 111.5) (mid 204.964466 110.035534) (end 203.5 106.5) (layer "Edge.Cuts") (width 0.15))
   (gr_line (start 208.5 31.5) (end 246 31.5) (layer "Edge.Cuts") (width 0.1))
+  (gr_text "HB9UF All-In-One-Box, Rev 1.0, (c) 2024 M. Weyland HB9FRV, based on work by skuep" (at 204.6 71.6 90) (layer "F.SilkS")
+    (effects (font (size 1 1) (thickness 0.2)))
+  )
   (dimension (type aligned) (layer "Dwgs.User")
     (pts (xy 203.5 111.5) (xy 215.375 111.5))

Commit message: Silk Screen artwork on pcb back
Parts:
- added G***: LOGO, symbols:hb9uf_logo, B.Cu at (234.2, 62.6)
- added SYM: Symbol_OSHW-Logo_SilkScreen_07Jul2012, symbols:Symbol_OSHW-Logo_SilkScreen, B.Cu at (244.2, 83.0)
- moved J2 1.08 mm to (241.1, 68.7)
- moved R14 0.96 mm to (243.2, 71.6)
Routing:
- net /NRST: track 75.9 -> 74.2 mm
- net /SWDIO: track 10.7 -> 9.74 mm
- net /SWO: track 13.4 -> 14.1 mm
- net /SWCLK: track 5.74 -> 6.31 mm
- net GND: track 38.8 -> 38.2 mm
Other:
- board text added: "All-In-One-Box"
- board text added: "By Matt Weyland (HB9FRV) based on work by skuep Rev 1.0, (c) 2024, MIT License"
- board text added: "HB9UF HB9UHF"

Commit message: Adding project URLs to back of PCB
Other:
- board text added: "https://github.com/HB9UF/AIOB"
- board text added: "https://github.com/skuep/AIOC"
Changed lines of the file:
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@@
   (gr_arc (start 208.5 111.5) (mid 204.964466 110.035534) (end 203.5 106.5) (layer "Edge.Cuts") (width 0.15))
   (gr_line (start 208.5 31.5) (end 246 31.5) (layer "Edge.Cuts") (width 0.1))
+  (gr_text "https://github.com/skuep/AIOC" (at 219.6 91.8) (layer "B.SilkS")
+    (effects (font (size 1 1) (thickness 0.2)) (justify mirror))
+  )
   (gr_text "All-In-One-Box\n" (at 208 77.4) (layer "B.SilkS")
     (effects (font (size 1.5 1.5) (thickness 0.3)) (justify right mirror))
   )
+  (gr_text "https://github.com/HB9UF/AIOB" (at 219.6 89.6) (layer "B.SilkS")
+    (effects (font (size 1 1) (thickness 0.2)) (justify mirror))
+  )
   (gr_text "HB9UF\nHB9UHF" (at 207 69.2) (layer "B.SilkS")

Commit message: Adding GND point for scope probe
Parts:
- added GND: GND, hb9uf:GND, F.Cu at (218.0, 57.2)
- added J5: GND, Connector_PinHeader_2.54mm:PinHeader_1x02_P2.54mm_Vertical, F.Cu at (221.0, 56.2)

Commit message: Adding LCSC (and some DIGIKEY) part numbers
Parts:
- R18, R19, R21, R22: value 24 -> 24R

Commit message: Improved placement of uC decoupling caps
Parts:
- moved C7 5.40 mm to (223.5, 72.4), turned to -90 degrees
- moved C15 1.00 mm to (217.8, 79.8)
- moved C9 1.00 mm to (217.8, 82.0)
Routing:
- net GND: track 38.2 -> 36.9 mm, vias 200 -> 207
- net /PTT1: track 11.5 -> 10.7 mm

Commit message: Adding TRRS pinout to silk screen
Routing:
- net GND: vias 207 -> 211
Other:
- board text added: "AUDIO"
- board text added: "CAT"
- board text added: "COS"
- board text added: "GND"
- board text added: "PTT"
- board text added: "TRX-IN"
- board text added: "TRX-OUT"
- board text added: "TRX-RX"
- board text added: "TRX-TX"
Changed lines of the file:
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@@
       ) (layer "B.SilkS") (width 0.1) (fill solid))
   )
+  (gr_line (start 226.137693 102.867386) (end 226.137693 102.867386) (layer "B.SilkS") (width 0.223652))
+  (gr_line (start 227.2 99.6) (end 226.196182 100.456285) (layer "B.SilkS") (width 0.223652))
+  (gr_line (start 228.454041 100.461748) (end 226.19268 100.461748) (layer "B.SilkS") (width 0.223652))
+  (gr_line (start 228.454041 100.461748) (end 228.454041 100.461748) (layer "B.SilkS") (width 0.223652))
+  (gr_poly
+    (pts
+      (xy 226.074947 108.018809)
+      (xy 226.074947 107.512632)
+      (xy 228.491242 107.512632)
+      (xy 228.491242 108.018809)
+    ) (layer "B.SilkS") (width 0) (fill solid))
+  (gr_line (start 228.430798 100.446414) (end 227.485389 99.59925) (layer "B.SilkS") (width 0.223652))
+  (gr_line (start 228.504917 109.49998) (end 228.504917 102.867386) (layer "B.SilkS") (width 0.223652))
+  (gr_line (start 227.2 99.6) (end 227.2 99.6) (layer "B.SilkS") (width 0.223652))
+  (gr_line (start 225.613952 109.578651) (end 225.613952 110.57634) (layer "B.SilkS") (width 0.201287))
+  (gr_line (start 228.504917 102.867386) (end 228.504917 102.867386) (layer "B.SilkS") (width 0.223652))
+  (gr_line (start 225.613952 109.578651) (end 225.613952 109.578651) (layer "B.SilkS") (width 0.201287))
+  (gr_line (start 226.19268 100.461748) (end 226.19268 100.461748) (layer "B.SilkS") (width 0.223652))
+  (gr_line (start 226.137693 102.867386) (end 226.140473 109.487063) (layer "B.SilkS") (width 0.223652))
+  (gr_line (start 228.226473 102.851172) (end 228.454041 100.461748) (layer "B.SilkS") (width 0.223652))
+  (gr_poly
+    (pts
+      (xy 226.095855 105.93115)
+      (xy 226.095855 105.424973)
+      (xy 228.51215 105.424973)
+      (xy 228.51215 105.93115)
+    ) (layer "B.SilkS") (width 0) (fill solid))
+  (gr_line (start 228.504917 102.867386) (end 226.137693 102.867386) (layer "B.SilkS") (width 0.223652))
+  (gr_line (start 227.485389 99.59925) (end 227.2 99.6) (layer "B.SilkS") (width 0.223652))
+  (gr_line (start 229.028656 109.578651) (end 225.613952 109.578651) (layer "B.SilkS") (width 0.201287))
+  (gr_line (start 229.028656 110.611363) (end 229.028656 109.578651) (layer "B.SilkS") (width 0.201287))
+  (gr_poly
+    (pts
+      (xy 226.118391 103.855172)
+      (xy 226.118391 103.348995)
+      (xy 228.534686 103.348995)
+      (xy 228.534686 103.855172)
+    ) (layer "B.SilkS") (width 0) (fill solid))
+  (gr_line (start 229.028656 109.578651) (end 229.028656 109.578651) (layer "B.SilkS") (width 0.201287))
+  (gr_line (start 226.19268 100.461748) (end 226.50007 102.860805) (layer "B.SilkS") (width 0.223652))
+  (gr_line (start 227.485389 99.59925) (end 227.485389 99.59925) (layer "B.SilkS") (width 0.223652))
   (gr_line (start 205 31.5) (end 205 111.5) (layer "Cmts.User") (width 0.15))
   (gr_line (start 249.5 31.5) (end 249.5 111.5) (layer "Cmts.User") (width 0.15))
@@
   (gr_arc (start 208.5 111.5) (mid 204.964466 110.035534) (end 203.5 106.5) (layer "Edge.Cuts") (width 0.15))
   (gr_line (start 208.5 31.5) (end 246 31.5) (layer "Edge.Cuts") (width 0.1))
+  (gr_text "CAT" (at 238.6 98) (layer "B.SilkS")
+    (effects (font (size 1.5 1.5) (thickness 0.3)) (justify mirror))
+  )
+  (gr_text "COS" (at 229 106.6) (layer "B.SilkS")
+    (effects (font (size 1 1) (thickness 0.2)) (justify right mirror))
+  )
+  (gr_text "TRX-IN" (at 225.556772 104.6) (layer "B.SilkS")
+    (effects (font (size 1 1) (thickness 0.2)) (justify left mirror))
+  )
+  (gr_text "TRX-RX" (at 229 101.8) (layer "B.SilkS")
+    (effects (font (size 1 1) (thickness 0.2)) (justify right mirror))
+  )
+  (gr_text "AUDIO" (at 214.8 98) (layer "B.SilkS")
+    (effects (font (size 1.5 1.5) (thickness 0.3)) (justify mirror))
+  )
   (gr_text "https://github.com/skuep/AIOC" (at 219.6 91.8) (layer "B.SilkS")
     (effects (font (size 1 1) (thickness 0.2)) (justify mirror))
@@
     (effects (font (size 1 1) (thickness 0.2)) (justify mirror))
   )
+  (gr_text "GND" (at 225.6 108.6) (layer "B.SilkS")
+    (effects (font (size 1 1) (thickness 0.2)) (justify left mirror))
+  )
   (gr_text "HB9UF\nHB9UHF" (at 207 69.2) (layer "B.SilkS")
     (effects (font (size 3 3) (thickness 0.6)) (justify right mirror))
+  )
+  (gr_text "GND" (at 229 108.6) (layer "B.SilkS")
+    (effects (font (size 1 1) (thickness 0.2)) (justify right mirror))
+  )
+  (gr_text "TRX-TX" (at 229 104.6) (layer "B.SilkS")
+    (effects (font (size 1 1) (thickness 0.2)) (justify right mirror))
+  )
+  (gr_text "TRX-OUT" (at 225.460917 101.8) (layer "B.SilkS")
+    (effects (font (size 1 1) (thickness 0.2)) (justify left mirror))
+  )
+  (gr_text "PTT" (at 225.6 106.6) (layer "B.SilkS")
+    (effects (font (size 1 1) (thickness 0.2)) (justify left mirror))
   )
   (gr_text "By Matt Weyland (HB9FRV)\nbased on work by skuep\nRev 1.0, (c) 2024, MIT License" (at 208 84.6) (layer "B.SilkS")
@@
   (via (at 220.2 65.4) (size 0.6) (drill 0.3) (layers "F.Cu" "B.Cu") (free) (net 1))
   (via (at 243.8 103.8) (size 0.6) (drill 0.3) (layers "F.Cu" "B.Cu") (free) (net 1))
+  (via (at 217.8 104.2) (size 0.8) (drill 0.4) (layers "F.Cu" "B.Cu") (free) (net 1))
   (via (at 210.8 75.55) (size 0.6) (drill 0.3) (layers "F.Cu" "B.Cu") (net 1))
   (via (at 214 48.2) (size 0.6) (drill 0.3) (layers "F.Cu" "B.Cu") (free) (net 1))
@@
   (via (at 233 85) (size 0.6) (drill 0.3) (layers "F.Cu" "B.Cu") (net 1))
   (via (at 206 79) (size 0.6) (drill 0.3) (layers "F.Cu" "B.Cu") (free) (net 1))
+  (via (at 213.4 104.2) (size 0.8) (drill 0.4) (layers "F.Cu" "B.Cu") (free) (net 1))
   (via (at 206.6 93) (size 0.6) (drill 0.3) (layers "F.Cu" "B.Cu") (free) (net 1))
   (via (at 208 74) (size 0.6) (drill 0.3) (layers "F.Cu" "B.Cu") (free) (net 1))
@@
   (via (at 245 91.5) (size 0.6) (drill 0.3) (layers "F.Cu" "B.Cu") (net 1))
   (via (at 206 87.8) (size 0.6) (drill 0.3) (layers "F.Cu" "B.Cu") (free) (net 1))
+  (via (at 218.6 100.2) (size 0.8) (drill 0.4) (layers "F.Cu" "B.Cu") (free) (net 1))
   (via (at 217.6 55) (size 0.6) (drill 0.3) (layers "F.Cu" "B.Cu") (free) (net 1))
   (via (at 217.2 64.8) (size 0.6) (drill 0.3) (layers "F.Cu" "B.Cu") (free) (net 1))
-  (via (at 226 104.8) (size 0.6) (drill 0.3) (layers "F.Cu" "B.Cu") (free) (net 1))
+  (via (at 225 105.6) (size 0.6) (drill 0.3) (layers "F.Cu" "B.Cu") (free) (net 1))
   (via (at 226.6 48.2) (size 0.6) (drill 0.3) (layers "F.Cu" "B.Cu") (free) (net 1))
   (via (at 243.8 79.4) (size 0.6) (drill 0.3) (layers "F.Cu" "B.Cu") (free) (net 1))
@@
   (via (at 228.8 64.8) (size 0.6) (drill 0.3) (layers "F.Cu" "B.Cu") (free) (net 1))
   (via (at 209 65.2) (size 0.6) (drill 0.3) (layers "F.Cu" "B.Cu") (free) (net 1))
+  (via (at 219.6 103.2) (size 0.8) (drill 0.4) (layers "F.Cu" "B.Cu") (free) (net 1))
   (via (at 206 86.4) (size 0.6) (drill 0.3) (layers "F.Cu" "B.Cu") (free) (net 1))
   (via (at 209.6 110.4) (size 0.6) (drill 0.3) (layers "F.Cu" "B.Cu") (free) (net 1))
@@
     )
   )
+  (group "" (id 7e0dbb2c-df5a-492b-80f8-8060034383db)
+    (members
+      041c688b-abb9-485c-b38f-9a9a7fca7f60
+      0ca670bd-7868-4fd8-a4c7-31a7c0d419cd
+      0d4017e9-3d19-4816-875b-db00f6681f52
+      534c5d96-c847-40d6-a305-2da84819b0e1
+      57398a82-60c0-40c1-ae35-b52467b46701
+      5f01045b-04b0-46b4-b5d6-f76fb04e5568
+      8b258ccd-ac03-40b8-9799-88cfd666e78d
+      a7feb3c0-4cd7-47a6-b300-c8f545729291
+      adf6283b-c1b0-4f64-8134-0474e5cbd6e2
+      ae5fb683-31ed-485b-88b9-501a09f1b84a
+      b58e76e8-cd4b-4238-a111-9bb30176e656
+      b9216d42-7fa9-49cb-b71c-2f60a03793aa
+      c4d01dce-ba4c-4f32-9e5c-6f4d99afe0ec
+      ccb32b51-e3f5-40c0-a5e4-fb6a29163a5f
+      d3d2fdb5-8a66-436a-8970-4fc87f50384a
+      d69405dd-6c61-4051-bcf9-7a9c2dc9766c
+      db99c40a-ff67-4a33-9efe-3bdfc36c03c9
+      e6692b46-b013-47f9-9787-18e4c1fae16a
+      e7c84213-22f9-4096-9a39-4f211205baa5
+      ea7d2f79-c444-4b50-9612-a24dd315260f
+      eb71b8b4-5a59-4bbf-aadf-7fd6d0b8e8d4
+      f5c3ba7a-cf71-4c3c-97d1-b5673ac4353c
+      fad65fbd-4e02-4f0e-a13b-28a37af14712
+    )
+  )
