File: kicad/k1-aioc/k1-aioc.kicad_pcb (KiCad board)
At the start: 2 copper layers, 47.5 x 80 mm, 62 parts, among them J1 12401832E402A, J2 Conn_01x07_Male, J3 AUDIO, J4 CAT, J5 GND, Q1 PZT2222A, Q2 PZT2222A, U1 TLV1117LV-33, U2 STM32F373CBTx, U3 TLV1117LV-33, U4 CRE1S0505SC, U5 ADUM3160, Y1 8MHz/20pF

Commit message: Re-running annotate to renumber
We shuffled and changed quite a number of parts in this branch, so it
makes sense to finally renumber the part annotations.
Parts:
- renumbered C15 to C1, C19 to C11, C11 to C12, C3 to C13, C6 to C14, C12 to C15, C14 to C16, C13 to C17, C4 to C18, C5 to C19, C1 to C2, C2 to C3, C18 to C4, C7 to C5, C16 to C6, C8 to C7, C17 to C8, FB2 to FB1, FB3 to FB2, FB1 to FB3, J5 to J2, J2 to J3, J3 to J4, J4 to J5, R18 to R1, R11 to R10, R17 to R11, R2 to R12, R8 to R13, R9 to R14, R16 to R15, R3 to R16, R4 to R17, R5 to R18, R10 to R19, R19 to R2, R13 to R20, R12 to R21, R15 to R22, R6 to R3, R14 to R4, R7 to R5, R20 to R6, R21 to R7, R22 to R8, R1 to R9, U4 to U1, U5 to U2, U2 to U3, U1 to U4, U3 to U5
